File: examples/FPGACONF/pcb/FPGACONF-02/010.sch (KiCad schematic (older format))
At the start: 33 parts, among them CN205 JST_SM04B-SRSS-TB, U201 STM32F730Z8T, U202 STM32F730V8T, X201 ASVTX-12-A-40.000MHZ-H10-T

Commit message: FPGACONF-02 schematics  support for SD-DDR (H743) test
Parts:
- removed U202: STM32F730V8T, zhtlab_SMD_QFP_QFN:TQFP-100_14x14mm_Pitch0.5mm, symbol STM32F730V8T
Connections:
- net VD_MCU: now also X201.1 (VCON)
- net MCU_PE2:QSPI_D2: now reaches U201.1 (PE2)
- net MCU_PA0:LED0: now reaches U201.34 (PA0)
- net MCU_PA1:LED1: now reaches U201.35 (PA1)
- net MCU_PA2:LED2: now reaches U201.36 (PA2)
- net MCU_PA3:LED3: now reaches U201.37 (PA3)
- net MCU_PA4:LED4: now reaches U201.40 (PA4)
- net MCU_PA5:LED5: now reaches U201.41 (PA5)
- net MCU_PA6:LED6: now reaches U201.42 (PA6)
- net MCU_PA7:LED7: now reaches U201.43 (PA7)
- net MCU_PB1:SDMMC1_VSEL33: now reaches U201.47 (PB1)
- net MCU_PB2:QSPI_CLK: now reaches U201.48 (PB2)
- net MCU_PD11:QSPI_D0: now reaches U201.82 (PD11)
- net MCU_PD12:QSPI_D1: now reaches U201.83 (PD12)
- net MCU_PD13:QSPI_D3: now reaches U201.84 (PD13)
- net MCU_PB0:FPGA_DONE renamed MCU_PB0:SDMMC1_PWREN
- net MCU_PB13:USB_ID renamed MCU_PB12:USB_ID
- net MCU_PB6:I2CS_SCL renamed MCU_PB6:I2CS_SCL_QSPI_CSX
- net MCU_PC3:SDMMC1_WP_X renamed MCU_PC3:FPGA_DONE
- net MCU_PC3:USB_VBUS_EN renamed MCU_PB13:USB_VBUS_EN
- net VD3P30_SD renamed VD_SDIO
- net VD3P30_USB renamed VD3P30
- no-connect marks 119 -> 50
Other:
- note added: "STM32F730, F733, F723: USBHS PHY, SDMMC SDR\nSTM32H750, H743: USBFS PHY, SDMMC DDR"
- note removed: "MCU"
