File: examples/FPGACONF/pcb/FPGACONF-02/022.sch (KiCad schematic (older format))
At the start: 20 parts, among them CN501 CN_10x2_D1.0mm_P2.54mm_TH, CN502 CN_07x2_D1.0mm_P2.54mm_TH, J501 SD_DM1B-DSF-PEJ

Commit message: FPGACONF-02 schematics  support for SD-DDR (H743) test
Parts:
- added C504: 0.1u, zhtlab_SMD_standard:RCL_1608m, symbol C0603
- added C505: 1u, zhtlab_SMD_standard:RCL_1608m, symbol C0603
- added C506: 0.01u, zhtlab_SMD_standard:RCL_1608m, symbol C0603
- added C507: 2.2u, zhtlab_SMD_standard:RCL_1608m, symbol C0603
- added Q501: RU1C001UN, zhtlab_SMD_standard:SC-85_2.0x2.0mm, symbol RU1C001UN
- added R515: 13k, zhtlab_SMD_standard:RCL_1608m, symbol R-1608M-5%
- added R516: 24k, zhtlab_SMD_standard:RCL_1608m, symbol R-1608M-5%
- added R517: 18k, zhtlab_SMD_standard:RCL_1608m, symbol R-1608M-5%
- added R518: 100k, zhtlab_SMD_standard:RCL_1608m, symbol R-1608M-5%
- added U501: MT25QL01GBBB8ESF-0SIT, zhtlab_SMD_standard:SOIC-16_10.3x10.3mm_Pitch1.27mm, symbol MT25QL01GBBB8ESF-0SIT
- added U502: TPS73001DBVR, zhtlab_SMD_standard:SOT-23-6_2.7x2.9mm_Pitch0.95mm, symbol TPS73001DBVR
- R509: value 0 -> 100k
- R511, R512, R513, R514: DNI DNI -> (none)
Connections:
- net VD_MCU: now also C504.2, U501.2 (VDD), U501.3 (RESET#)
- net MCU_PB0:FPGA_DONE renamed MCU_PC3:FPGA_DONE
- net MCU_PC3:SDMMC1_WP_X: no longer names the net of R508.1
- net VD3P30_SD renamed VD_SDIO
- net VD_SDIO: now also C507.2, R517.2, U502.6 (OUT); no longer C501.2, J501.4 (VDD), R509.1
- new net: C506.2, U502.4 (NR)
- new net: R515.2, R517.1, U502.5 (FB)
- new net: Q501.3, R515.1, R516.2
- new net MCU_PB0:SDMMC1_PWREN: R518.2, U502.3 (EN)
- new net MCU_PB1:SDMMC1_VSEL33: Q501.1, R509.1
- new net MCU_PB2:QSPI_CLK: U501.16 (CLK)
- new net MCU_PB6:I2CS_SCL_QSPI_CSX: U501.7 (CS#)
- new net MCU_PD11:QSPI_D0: U501.15 (DQ0/DI)
- new net MCU_PD12:QSPI_D1: U501.8 (DQ1/DO)
- new net MCU_PD13:QSPI_D3: U501.1 (DQ3/HOLD#)
- new net MCU_PE2:QSPI_D2: U501.9 (DQ2/WP#)
- new net VD3P30: C501.2, C505.2, J501.4 (VDD), U502.1 (IN)
- no-connect marks 2 -> 10
Other:
- note added: "QSPI FLASH ROM"
- note added: "R1"
- note added: "R2"
- note added: "R2(3.3V) = 18k / (2.9/1.225 - 1) = 13.16k\nR2(1.8V) = 18k / (1.8/1.225 - 1) = 38.35k\n\nVout(3.3V) = 1.225 * (18k / 13.0k + 1) = 2.92V\nVout(1.8V) = 1.225 * (18k / 37.0k + 1) = 1.82V"
